Commit message: WIP

File: AiRobot/training/filename.urdf (robot description, URDF)
Before this commit: robot my_bot, 17 links, 16 joints
Links:
- removed link 0_0
- removed link 0_1
- removed link 0_2
- removed link 0_3
- removed link 1_0
- removed link 1_1
- removed link 1_2
- removed link 1_3
- removed link 2_0
- removed link 2_1
- removed link 2_2
- removed link 2_3
- removed link 3_0
- removed link 3_1
- removed link 3_2
- removed link 3_3
Joints:
- removed joint 0_0
- removed joint 0_1
- removed joint 0_2
- removed joint 0_3
- removed joint 1_0
- removed joint 1_1
- removed joint 1_2
- removed joint 1_3
- removed joint 2_0
- removed joint 2_1
- removed joint 2_2
- removed joint 2_3
- removed joint 3_0
- removed joint 3_1
- removed joint 3_2
- removed joint 3_3
